File: KiCad-Shield-Uno-FlexSensor/KiCad-Shield-Uno-FlexSensor.kicad_pcb (KiCad board)
At the start: 2 copper layers, 68.6 x 53.3 mm, 8 parts, among them J1 Power, J2 Digital/PWM, J3 Analog, J4 Digital/PWM

Commit message: Shield UNO pour démarrage projet FlexSensor
Connections:
- J1 pad 2: /IOREF -> unconnected-(J1-Pin_2-Pad2)
- J1 pad 3: /~{RESET} -> unconnected-(J1-Pin_3-Pad3)
- J2 pad 1: /SCL/A5 -> unconnected-(J2-Pin_1-Pad1)
- J2 pad 10: /8 -> unconnected-(J2-Pin_10-Pad10)
- J2 pad 2: /SDA/A4 -> unconnected-(J2-Pin_2-Pad2)
- J2 pad 3: /AREF -> unconnected-(J2-Pin_3-Pad3)
- J2 pad 5: /13 -> unconnected-(J2-Pin_5-Pad5)
- J2 pad 6: /12 -> unconnected-(J2-Pin_6-Pad6)
- J2 pad 7: /*11 -> unconnected-(J2-Pin_7-Pad7)
- J2 pad 8: /*10 -> unconnected-(J2-Pin_8-Pad8)
- J2 pad 9: /*9 -> unconnected-(J2-Pin_9-Pad9)
- J3 pad 1: /A0 -> unconnected-(J3-Pin_1-Pad1)
- J3 pad 2: /A1 -> unconnected-(J3-Pin_2-Pad2)
- J3 pad 3: /A2 -> unconnected-(J3-Pin_3-Pad3)
- J3 pad 4: /A3 -> unconnected-(J3-Pin_4-Pad4)
- J3 pad 5: /SDA/A4 -> unconnected-(J3-Pin_5-Pad5)
- J3 pad 6: /SCL/A5 -> unconnected-(J3-Pin_6-Pad6)
- J4 pad 1: /7 -> unconnected-(J4-Pin_1-Pad1)
- J4 pad 2: /*6 -> unconnected-(J4-Pin_2-Pad2)
- J4 pad 3: /*5 -> unconnected-(J4-Pin_3-Pad3)
- J4 pad 4: /4 -> unconnected-(J4-Pin_4-Pad4)
- J4 pad 5: /*3 -> unconnected-(J4-Pin_5-Pad5)
- J4 pad 6: /2 -> unconnected-(J4-Pin_6-Pad6)
- J4 pad 7: /TX/1 -> unconnected-(J4-Pin_7-Pad7)
- J4 pad 8: /RX/0 -> unconnected-(J4-Pin_8-Pad8)
